File: usb-ttl.kicad_pcb (KiCad board)
At the start: 2 copper layers, 25 x 16 mm, 9 parts, among them J1 USB_A, J2 Conn_01x05, U1 CH330N

Commit message: update
Routing:
- net +5V: track 34.6 -> 35.5 mm
Changed lines of the file:
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@@
       (effects (font (size 1 1) (thickness 0.15)))
     )
+    (fp_line (start -4.85 -6.145) (end -3.8 -6.145) (layer "F.SilkS") (width 0.12))
+    (fp_line (start -8.02 -4.4) (end -8.775 -4.4) (layer "F.SilkS") (width 0.12))
+    (fp_line (start -8.02 -4.4) (end -8.02 4.4) (layer "F.SilkS") (width 0.12))
     (fp_line (start -4.85 6.145) (end -3.8 6.145) (layer "F.SilkS") (width 0.12))
-    (fp_line (start -4.85 -6.145) (end -3.8 -6.145) (layer "F.SilkS") (width 0.12))
-    (fp_line (start -8.02 -4.4) (end -8.02 4.4) (layer "F.SilkS") (width 0.12))
-    (fp_line (start -8.02 -4.4) (end -8.775 -4.4) (layer "F.SilkS") (width 0.12))
     (fp_line (start -3.8 6.025) (end -3.8 -6.025) (layer "Dwgs.User") (width 0.1))
     (fp_line (start -4.65 7.15) (end -4.65 6.52) (layer "F.CrtYd") (width 0.05))
+    (fp_line (start -4.65 -6.52) (end 11.4 -6.52) (layer "F.CrtYd") (width 0.05))
+    (fp_line (start -11.4 -4.55) (end -9.15 -4.55) (layer "F.CrtYd") (width 0.05))
+    (fp_line (start -9.15 7.15) (end -4.65 7.15) (layer "F.CrtYd") (width 0.05))
+    (fp_line (start -9.15 4.55) (end -9.15 7.15) (layer "F.CrtYd") (width 0.05))
+    (fp_line (start -4.65 -6.52) (end -4.65 -7.15) (layer "F.CrtYd") (width 0.05))
+    (fp_line (start -11.4 4.55) (end -9.15 4.55) (layer "F.CrtYd") (width 0.05))
+    (fp_line (start -11.4 4.55) (end -11.4 -4.55) (layer "F.CrtYd") (width 0.05))
+    (fp_line (start -9.15 -7.15) (end -9.15 -4.55) (layer "F.CrtYd") (width 0.05))
+    (fp_line (start -4.65 6.52) (end 11.4 6.52) (layer "F.CrtYd") (width 0.05))
     (fp_line (start 11.4 6.52) (end 11.4 -6.52) (layer "F.CrtYd") (width 0.05))
-    (fp_line (start -11.4 -4.55) (end -9.15 -4.55) (layer "F.CrtYd") (width 0.05))
-    (fp_line (start -4.65 6.52) (end 11.4 6.52) (layer "F.CrtYd") (width 0.05))
-    (fp_line (start -4.65 -6.52) (end 11.4 -6.52) (layer "F.CrtYd") (width 0.05))
-    (fp_line (start -4.65 -6.52) (end -4.65 -7.15) (layer "F.CrtYd") (width 0.05))
-    (fp_line (start -9.15 4.55) (end -9.15 7.15) (layer "F.CrtYd") (width 0.05))
-    (fp_line (start -9.15 -7.15) (end -9.15 -4.55) (layer "F.CrtYd") (width 0.05))
-    (fp_line (start -11.4 4.55) (end -11.4 -4.55) (layer "F.CrtYd") (width 0.05))
-    (fp_line (start -9.15 7.15) (end -4.65 7.15) (layer "F.CrtYd") (width 0.05))
-    (fp_line (start -11.4 4.55) (end -9.15 4.55) (layer "F.CrtYd") (width 0.05))
     (fp_line (start -9.15 -7.15) (end -4.65 -7.15) (layer "F.CrtYd") (width 0.05))
+    (fp_line (start -10.4 3.75) (end -7.9 3.75) (layer "F.Fab") (width 0.1))
+    (fp_line (start -10.4 -0.75) (end -7.9 -0.75) (layer "F.Fab") (width 0.1))
+    (fp_line (start -10.4 3.75) (end -10.4 3.25) (layer "F.Fab") (width 0.1))
+    (fp_line (start -10.4 -3.75) (end -7.9 -3.75) (layer "F.Fab") (width 0.1))
+    (fp_line (start -10.4 1.25) (end -7.9 1.25) (layer "F.Fab") (width 0.1))
+    (fp_line (start -10.4 -3.25) (end -7.9 -3.25) (layer "F.Fab") (width 0.1))
+    (fp_line (start -7.9 -6.025) (end 10.9 -6.025) (layer "F.Fab") (width 0.1))
+    (fp_line (start -7.25 -4) (end -7.25 -3.05) (layer "F.Fab") (width 0.1))
+    (fp_line (start -7.9 6.025) (end -7.9 -6.025) (layer "F.Fab") (width 0.1))
     (fp_line (start 10.9 6.025) (end 10.9 -6.025) (layer "F.Fab") (width 0.1))
-    (fp_line (start -10.4 3.75) (end -7.9 3.75) (layer "F.Fab") (width 0.1))
     (fp_line (start -10.4 -1.25) (end -7.9 -1.25) (layer "F.Fab") (width 0.1))
-    (fp_line (start -7.25 -4) (end -7.25 -3.05) (layer "F.Fab") (width 0.1))
-    (fp_line (start -10.4 -0.75) (end -7.9 -0.75) (layer "F.Fab") (width 0.1))
-    (fp_line (start -7.9 -6.025) (end 10.9 -6.025) (layer "F.Fab") (width 0.1))
-    (fp_line (start -10.4 -3.25) (end -7.9 -3.25) (layer "F.Fab") (width 0.1))
-    (fp_line (start -7.75 -3.5) (end -7.25 -4) (layer "F.Fab") (width 0.1))
+    (fp_line (start -10.4 3.25) (end -7.9 3.25) (layer "F.Fab") (width 0.1))
     (fp_line (start -7.9 6.025) (end 10.9 6.025) (layer "F.Fab") (width 0.1))
     (fp_line (start -10.4 -3.25) (end -10.4 -3.75) (layer "F.Fab") (width 0.1))
+    (fp_line (start -10.4 0.75) (end -7.9 0.75) (layer "F.Fab") (width 0.1))
     (fp_line (start -10.4 1.25) (end -10.4 0.75) (layer "F.Fab") (width 0.1))
-    (fp_line (start -7.9 6.025) (end -7.9 -6.025) (layer "F.Fab") (width 0.1))
-    (fp_line (start -10.4 1.25) (end -7.9 1.25) (layer "F.Fab") (width 0.1))
-    (fp_line (start -10.4 3.75) (end -10.4 3.25) (layer "F.Fab") (width 0.1))
-    (fp_line (start -10.4 -3.75) (end -7.9 -3.75) (layer "F.Fab") (width 0.1))
-    (fp_line (start -10.4 3.25) (end -7.9 3.25) (layer "F.Fab") (width 0.1))
     (fp_line (start -10.4 -0.75) (end -10.4 -1.25) (layer "F.Fab") (width 0.1))
-    (fp_line (start -10.4 0.75) (end -7.9 0.75) (layer "F.Fab") (width 0.1))
     (fp_line (start -7.75 -3.5) (end -7.25 -3) (layer "F.Fab") (width 0.1))
+    (fp_line (start -7.75 -3.5) (end -7.25 -4) (layer "F.Fab") (width 0.1))
+    (fp_circle (center -6.9 -2.3) (end -6.9 -2.8) (layer "F.Fab") (width 0.1) (fill none))
     (fp_circle (center -6.9 2.3) (end -6.9 2.8) (layer "F.Fab") (width 0.1) (fill none))
-    (fp_circle (center -6.9 -2.3) (end -6.9 -2.8) (layer "F.Fab") (width 0.1) (fill none))
+    (pad "" np_thru_hole circle (at -6.9 2.3 180) (size 1.1 1.1) (drill 1.1) (layers *.Cu *.Mask))
     (pad "" np_thru_hole circle (at -6.9 -2.3 180) (size 1.1 1.1) (drill 1.1) (layers *.Cu *.Mask))
-    (pad "" np_thru_hole circle (at -6.9 2.3 180) (size 1.1 1.1) (drill 1.1) (layers *.Cu *.Mask))
     (pad "1" smd rect (at -9.65 -3.5 180) (size 2.5 1.1) (layers "F.Cu" "F.Paste" "F.Mask")
       (net 1 "+5V") (pinfunction "VBUS") (pintype "power_in"))
@@
     (pad "5" thru_hole oval (at -6.9 5.7 180) (size 3.5 1.9) (drill oval 2.5 0.9) (layers *.Cu *.Mask)
       (net 2 "GND") (pinfunction "Shield") (pintype "passive"))
-    (model "/Users/niksun/Documents/KiCad/6.0/3dmodels/USB_A_CNCTech/USB_A_CNCTech_1001-011-01101_Horizontal.wrl"
+    (model "${KICAD6_3DMODEL_DIR}/Connector_USB.3dshapes/USB_A_CNCTech_1001-011-01101_Horizontal.wrl"
       (offset (xyz 0 0 0))
       (scale (xyz 1 1 1))
@@
   (segment (start 175.975 97.275) (end 176 97.3) (width 1) (layer "F.Cu") (net 1))
   (segment (start 175.2545 93.705) (end 175.975 93.705) (width 0.5) (layer "F.Cu") (net 1))
-  (via (at 174.5 92.9) (size 0.7) (drill 0.4) (layers "F.Cu" "B.Cu") (net 1))
+  (via (at 173.9 92.4) (size 0.7) (drill 0.4) (layers "F.Cu" "B.Cu") (net 1))
   (via (at 178.5 86.5) (size 0.7) (drill 0.4) (layers "F.Cu" "B.Cu") (net 1))
-  (segment (start 174.5 93) (end 176.5 93) (width 0.5) (layer "B.Cu") (net 1))
-  (segment (start 176.5 93) (end 178.4 91.099999) (width 0.5) (layer "B.Cu") (net 1))
-  (segment (start 178.4 91.099999) (end 178.4 86.6) (width 0.5) (layer "B.Cu") (net 1))
-  (segment (start 178.4 86.6) (end 178.5 86.5) (width 0.5) (layer "B.Cu") (net 1))
+  (segment (start 178.5 91) (end 178.5 86.5) (width 0.5) (layer "B.Cu") (net 1))
+  (segment (start 176.44952 93.05048) (end 178.5 91) (width 0.5) (layer "B.Cu") (net 1))
+  (segment (start 174.55048 93.05048) (end 173.9 92.4) (width 0.5) (layer "B.Cu") (net 1))
+  (segment (start 176.44952 93.05048) (end 174.55048 93.05048) (width 0.5) (layer "B.Cu") (net 1))
   (segment (start 175.975 88.2) (end 175.975 89.895) (width 0.5) (layer "F.Cu") (net 3))
   (segment (start 181.7975 92.6125) (end 183.725 94.54) (width 0.5) (layer "F.Cu") (net 4))
@@
   (segment (start 165.85 93) (end 166.55 93) (width 0.28) (layer "F.Cu") (net 8))
   (segment (start 166.55 93) (end 167.334 92.216) (width 0.28) (layer "F.Cu") (net 8))
-  (segment (start 170.606001 90.313999) (end 171.025 89.895) (width 0.28) (layer "F.Cu") (net 9))
+  (segment (start 170.086098 89.895) (end 171.025 89.895) (width 0.28) (layer "F.Cu") (net 9))
+  (segment (start 167.334 91.784) (end 168.197098 91.784) (width 0.28) (layer "F.Cu") (net 9))
+  (segment (start 166.55 91) (end 167.334 91.784) (width 0.28) (layer "F.Cu") (net 9))
+  (segment (start 168.197098 91.784) (end 170.086098 89.895) (width 0.28) (layer "F.Cu") (net 9))
   (segment (start 165.85 91) (end 166.55 91) (width 0.28) (layer "F.Cu") (net 9))
-  (segment (start 167.334 91.784) (end 168.193588 91.784) (width 0.28) (layer "F.Cu") (net 9))
-  (segment (start 169.663589 90.313999) (end 170.606001 90.313999) (width 0.28) (layer "F.Cu") (net 9))
-  (segment (start 166.55 91) (end 167.334 91.784) (width 0.28) (layer "F.Cu") (net 9))
-  (segment (start 168.193588 91.784) (end 169.663589 90.313999) (width 0.28) (layer "F.Cu") (net 9))
   (segment (start 171.025 93.705) (end 173.095 93.705) (width 0.5) (layer "F.Cu") (net 10))
   (segment (start 173.095 93.705) (end 173.1 93.7) (width 0.5) (layer "F.Cu") (net 10))
   (via (at 173.1 93.7) (size 0.7) (drill 0.4) (layers "F.Cu" "B.Cu") (net 10))
-  (segment (start 176.718559 93.7) (end 179.04952 91.369039) (width 0.5) (layer "B.Cu") (net 10))
-  (segment (start 179.04952 91.369039) (end 179.04952 88.85048) (width 0.5) (layer "B.Cu") (net 10))
+  (segment (start 179.149519 90.730959) (end 179.14952 88.75048) (width 0.5) (layer "B.Cu") (net 10))
+  (segment (start 176.718559 93.7) (end 179.14952 91.269039) (width 0.5) (layer "B.Cu") (net 10))
+  (segment (start 179.14952 88.75048) (end 180.98 86.92) (width 0.5) (layer "B.Cu") (net 10))
+  (segment (start 179.14952 91.269039) (end 179.149519 90.730959) (width 0.5) (layer "B.Cu") (net 10))
+  (segment (start 173.1 93.7) (end 176.718559 93.7) (width 0.5) (layer "B.Cu") (net 10))
   (segment (start 180.98 86.92) (end 183.725 86.92) (width 0.5) (layer "B.Cu") (net 10))
-  (segment (start 179.04952 88.85048) (end 180.98 86.92) (width 0.5) (layer "B.Cu") (net 10))
-  (segment (start 173.1 93.7) (end 176.718559 93.7) (width 0.5) (layer "B.Cu") (net 10))
   (zone (net 2) (net_name "GND") (layer "F.Cu") (hatch edge 0.508)
     (connect_pads (clearance 0.15))
